File: eagle/sensor.sch (EAGLE design)
At the start: 8 parts, among them IC1 LM358N, X1 1503_02, X2 0-Vcc

Commit message: reduce board size
Parts:
- D1: value 1N4148DO35-10 -> 1N4148
Changed lines of the file:
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@@
 <parts>
 <part name="IC1" library="linear" deviceset="LM358" device="N"/>
-<part name="D1" library="diode" deviceset="1N4148" device="DO35-10"/>
+<part name="D1" library="diode" deviceset="1N4148" device="DO35-10" value="1N4148"/>
 <part name="R1" library="rcl" deviceset="R-US_" device="0207/10" value="100k"/>
 <part name="R2" library="rcl" deviceset="R-US_" device="0207/10" value="39k"/>
